Commit message: Changed LD to AMR throughout the package and documentation

File: src/amr_visualisation/urdf/AMR_Platform.urdf (robot description, URDF)
Before this commit: robot LD_Platform, 8 links, 7 joints
Links:
- link main_body: geometry collision mesh filename=package://amr_visualisation/meshes/AMR_Platform.STL; visual mesh filename=package://amr_visualisation/meshes/AMR_Platform.STL
